Commit message: [1.3.0] Added base_footprint link to robot model
Added a base_footprint link to the robot model, making it more compatible with
third-party packages.

Signed-off-by: Helio Perroni Filho <xperroni@gmail.com>

File: urdf/ugv02.xacro (robot description, xacro)
@@ -131,3 +131,8 @@
     z="${ground_clearance + 0.5 * body_height}"
   />
+  <link name="base_footprint"/>
+  <xacro:joint_fixed
+    parent="base_link"
+    child="base_footprint"
+  />
 </robot>
